Commit message: module 5: add RViz configuration and static bridge parameters for simulation environment

File: src/household_robot_simulation/urdf/custom_robot.urdf (robot description, URDF)
Before this commit: robot custom_robot, 6 links, 5 joints
Links:
- added link camera_link, mass 0.05; collision box size=0.02 0.04 0.02; visual box size=0.02 0.04 0.02
- added link camera_link_optical
- added link imu_link, mass 0.01; collision box size=0.02 0.02 0.01; visual box size=0.02 0.02 0.01
- added link lidar_link, mass 0.1; collision cylinder length=0.04 radius=0.04; visual cylinder length=0.04 radius=0.04
- link base_link: geometry collision cylinder length=0.15 radius=0.2; visual box size=0.06 0.04 0.02
Joints:
- added joint camera_joint: type fixed, parent base_link, child camera_link, origin xyz=0.2 0 0.1 rpy=0 0 0
- added joint camera_optical_joint: type fixed, parent camera_link, child camera_link_optical, origin xyz=0 0 0 rpy=-1.57079632679 0 -1.57079632679
- added joint imu_joint: type fixed, parent base_link, child imu_link, origin xyz=0 0 0.08 rpy=0 0 0
- added joint lidar_joint: type fixed, parent base_link, child lidar_link, origin xyz=0 0 0.15 rpy=0 0 0

Commit message: module : 7

File: src/household_robot_simulation/urdf/custom_robot.urdf (robot description, URDF)
Before this commit: robot custom_robot, 10 links, 9 joints
Joints:
- joint left_wheel_joint: limit (none) -> effort=1.5 velocity=10.0
- joint right_wheel_joint: limit (none) -> effort=1.5 velocity=10.0
